File: stratosteam/gps.kicad_sch (KiCad schematic)
At the start: 1 part

Commit message: pcb
Connections:
- net UART_TX is gone; now on net UART_RX: U1. (GND)
Changed lines of the file:
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@@
-		)
-	)
-	(global_label "UART_TX"
-		(shape input)
-		(at 163.83 53.34 0)
-		(fields_autoplaced yes)
-		(effects
-			(font
-				(size 1.27 1.27)
-			)
-			(justify left)
-		)
-		(property "Intersheetrefs" "${INTERSHEET_REFS}"
-			(at 174.6166 53.34 0)
-			(hide yes)
-			(show_name no)
-			(do_not_autoplace no)
-			(effects
-				(font
-					(size 1.27 1.27)
-				)
-				(justify left)
-			)
 		)
 	)
