File: stratosteam/jonosfera.kicad_sch (KiCad schematic)
At the start: 10 parts, among them Q1 RD06HHF1, U3 AD9833, U4 LPF-B0R3, Y1 XO32

Commit message: pcb
Parts:
- removed C1, C3, C4, C6: 100n, Capacitor_SMD:C_0603_1608Metric_Pad1.08x0.95mm_HandSolder, symbol Device:C
- removed C2, C5: 10u, Capacitor_SMD:C_0603_1608Metric_Pad1.08x0.95mm_HandSolder, symbol Device:C
- removed Q1: RD06HHF1, Package_TO_SOT_THT:TO-220-3_Vertical, symbol Transistor_FET:IRF540N
- removed U3: AD9833, AD9833:SOP50P490X110-10N, symbol AD9833:AD9833
- removed U4: LPF-B0R3, RF_Mini-Circuits:Mini-Circuits_HZ1198_LandPatternPL-247, symbol RF_Filter:LPF-B0R3
- removed Y1: XO32, Oscillator:Oscillator_SMD_EuroQuartz_XO32-4Pin_3.2x2.5mm_RotB_HandSoldering, symbol Oscillator:XO32
